File: hardware/temperature.kicad_pcb (KiCad board)
At the start: 2 copper layers, 15 x 25 mm, 14 parts, among them P1 CON-SENSOR, U1 M24C64, U2 TMP102, U3 DRILL, U4 DRILL, U5 DRILL, U6 DRILL

Commit message: Add 3d information (final)
Parts:
- C1, C2: footprint 0603 -> kicad-libraries:C0603
- Fiducial_Mark (x2): footprint Fiducial_Mark -> kicad-libraries:Fiducial_Mark
- P1: footprint CON-SENSOR -> kicad-libraries:CON-SENSOR
- Ref**: footprint Logo_31x31 -> kicad-libraries:Logo_31x31
- U1: footprint TSSOP8 -> kicad-libraries:TSSOP8
- U3, U4, U5, U6: footprint DRILL_NP -> kicad-libraries:DRILL_NP
- VAL: footprint CE_5mm -> kicad-libraries:CE_5mm
- VAL: footprint WEEE_7mm -> kicad-libraries:WEEE_7mm
- turned VAL to 180 degrees
Connections:
- P1 pad 1: (no net) -> Net-(P1-Pad1)
- P1 pad 10: (no net) -> Net-(P1-Pad10)
- P1 pad 8: (no net) -> Net-(P1-Pad8)
- P1 pad 9: (no net) -> Net-(P1-Pad9)
- U1 pad 7: (no net) -> Net-(U1-Pad7)
